File: board/MCU.sch (KiCad schematic (older format))
At the start: 13 parts, among them J1 ICSP, U1 PIC16F15345-IP, U2 MAX232I, Y1 8MHz

Commit message: Add button 2, LEDs, TVS diode
* Add button 2; rewire to match the prototype
* Add a TVS diode across the 12V rail; value TBD
* Rework power nets into the power sheet; don't use the globals
  inside the sheet, expose the rails as pins.
* Move power protection inside the power sheet.
* Add power LEDs
Connections:
- net BUT2_UP: now reaches U1.14 (RC2)
- net BUT2_DN: now reaches U1.7 (RC3)
- net BUTTON_DN renamed BUT1_DN
- net BUTTON_UP renamed BUT1_UP
Changed lines of the file:
@@
 Sheet 2 4
 Title "Projector Screen Controller"
-Date ""
+Date "2019-08-31"
 Rev "0.1"
 Comp "Chris Luke"
-Comment1 ""
+Comment1 "https://github.com/flirbleoss/projector-screen-controller"
 Comment2 ""
 Comment3 ""
@@
 	1950 4400 2500 4400
 Text HLabel 7150 2700 1    50   Input ~ 0
-BUTTON_UP
+BUT1_UP
 Text HLabel 7250 2700 1    50   Input ~ 0
-BUTTON_DN
+BUT1_DN
 Wire Wire Line
 	7150 2700 7150 3500
@@
 	850  3900 2500 3900
 Connection ~ 850  4250
+Text HLabel 7350 2700 1    50   Input ~ 0
+BUT2_UP
+Text HLabel 7450 2700 1    50   Input ~ 0
+BUT2_DN
+Wire Wire Line
+	7350 2700 7350 3700
+Wire Wire Line
+	7350 3700 6900 3700
+Wire Wire Line
+	7450 2700 7450 3800
+Wire Wire Line
+	7450 3800 6900 3800
 $EndSCHEMATC

Commit message: Minor layout tweaks, component updates
* Add an MCU driven status LED
* Update LED current limit resistor values
* Minor trace tweaks for clearance
* Based on empirical measurements of rev 0.1 board, adjust the location of the
  board mounting holes.
Parts:
- added D12: LED, LEDs:LED_D3.0mm, symbol Device:LED
- added R8: 330R, Resistors_THT:R_Axial_DIN0207_L6.3mm_D2.5mm_P10.16mm_Horizontal, symbol Device:R
Connections:
- net GND: now also D12.1 (K)
- net at U1.17 (RA2): now also R8.1
- new net: D12.2 (A), R8.2
Changed lines of the file:
@@
 Wire Wire Line
 	7450 3800 6900 3800
+$Comp
+L Device:LED D12
+U 1 1 5D733225
+P 2300 5600
+F 0 "D12" V 2339 5483 50  0000 R CNN
+F 1 "LED" V 2248 5483 50  0000 R CNN
+F 2 "LEDs:LED_D3.0mm" H 2300 5600 50  0001 C CNN
+F 3 "~" H 2300 5600 50  0001 C CNN
+	1    2300 5600
+	0    -1   -1   0
+$EndComp
+$Comp
+L Device:R R8
+U 1 1 5D73555C
+P 2300 5250
+F 0 "R8" H 2370 5296 50  0000 L CNN
+F 1 "330R" H 2370 5205 50  0000 L CNN
+F 2 "Resistors_THT:R_Axial_DIN0207_L6.3mm_D2.5mm_P10.16mm_Horizontal" V 2230 5250 50  0001 C CNN
+F 3 "~" H 2300 5250 50  0001 C CNN
+	1    2300 5250
+	1    0    0    -1
+$EndComp
+$Comp
+L power:GND #PWR0111
+U 1 1 5D735E3D
+P 2300 5950
+F 0 "#PWR0111" H 2300 5700 50  0001 C CNN
+F 1 "GND" H 2305 5777 50  0000 C CNN
+F 2 "" H 2300 5950 50  0001 C CNN
+F 3 "" H 2300 5950 50  0001 C CNN
+	1    2300 5950
+	1    0    0    -1
+$EndComp
+Wire Wire Line
+	2500 3700 2300 3700
+Wire Wire Line
+	2300 3700 2300 5100
+Wire Wire Line
+	2300 5400 2300 5450
+Wire Wire Line
+	2300 5750 2300 5950
 $EndSCHEMATC

Commit message: Split the 5v and 12v ground paths
* To control the return path for (noisy) relay current, split the grounds for
  the 12v and 5v sections.
* The grounds are joined by bridges (solder pads) placed adjacent to the 5v
  regulator, on both layers.
* The gound plane is split in two; conveniently the 12v vs 5v components were
  already well placed to make this straightforward.
* 12v power LED uses the 5v ground to simplify routing.
* Add dummy power flags for ERC
Other:
- note added: "Optional programming\nheader components"
Changed lines of the file:
@@
 Sheet 2 4
 Title "Projector Screen Controller"
-Date "2019-09-02"
+Date "2019-09-07"
 Rev "0.2"
 Comp "Flirble Open Source"
@@
 Wire Wire Line
 	2300 5750 2300 5950
+Text Notes 2300 2000 1    50   ~ 0
+Optional programming\nheader components
 $EndSCHEMATC

Commit message: Update all footprints to KiCad 5 paths
* All footprints updated.
* 3D models for the relays seem to be missing from KiCad, however, so I
  have a copy in my personal library. Mostly cosmetic.
Parts:
- C1, C2, C3, C4, C5, C6, C7, C8: footprint Capacitors_THT:C_Disc_D5.0mm_W2.5mm_P2.50mm -> Capacitor_THT:C_Disc_D5.0mm_W2.5mm_P2.50mm
- D12: footprint LEDs:LED_D3.0mm -> LED_THT:LED_D3.0mm
- R1, R8: footprint Resistors_THT:R_Axial_DIN0207_L6.3mm_D2.5mm_P10.16mm_Horizontal -> Resistor_THT:R_Axial_DIN0207_L6.3mm_D2.5mm_P10.16mm_Horizontal
- U1: footprint Housings_DIP:DIP-20_W7.62mm_LongPads -> Package_DIP:DIP-20_W7.62mm_LongPads
- U2: footprint Housings_DIP:DIP-16_W7.62mm_LongPads -> Package_DIP:DIP-16_W7.62mm_LongPads
- Y1: footprint Crystals:Crystal_HC49-4H_Vertical -> Crystal:Crystal_HC49-4H_Vertical
Changed lines of the file:
@@
 F 0 "U2" H 8650 4950 50  0000 C CNN
 F 1 "MAX232I" H 8900 4950 50  0000 C CNN
-F 2 "Housings_DIP:DIP-16_W7.62mm_LongPads" H 9250 2850 50  0001 L CNN
+F 2 "Package_DIP:DIP-16_W7.62mm_LongPads" H 9250 2850 50  0001 L CNN
 F 3 "http://www.ti.com/lit/ds/symlink/max232.pdf" H 9200 4000 50  0001 C CNN
 	1    9200 3900
@@
 F 0 "C1" H 4365 5246 50  0000 L CNN
 F 1 "0.1uF" H 4365 5155 50  0000 L CNN
-F 2 "Capacitors_THT:C_Disc_D5.0mm_W2.5mm_P2.50mm" H 4288 5050 50  0001 C CNN
+F 2 "Capacitor_THT:C_Disc_D5.0mm_W2.5mm_P2.50mm" H 4288 5050 50  0001 C CNN
 F 3 "~" H 4250 5200 50  0001 C CNN
 	1    4250 5200
@@
 F 0 "C2" H 8865 5446 50  0000 L CNN
 F 1 "1uF" H 8865 5355 50  0000 L CNN
-F 2 "Capacitors_THT:C_Disc_D5.0mm_W2.5mm_P2.50mm" H 8788 5250 50  0001 C CNN
+F 2 "Capacitor_THT:C_Disc_D5.0mm_W2.5mm_P2.50mm" H 8788 5250 50  0001 C CNN
 F 3 "~" H 8750 5400 50  0001 C CNN
 	1    8750 5400
@@
 F 0 "Y1" H 1000 4518 50  0000 C CNN
 F 1 "8MHz" H 1000 4427 50  0000 C CNN
-F 2 "Crystals:Crystal_HC49-4H_Vertical" H 1000 4250 50  0001 C CNN
+F 2 "Crystal:Crystal_HC49-4H_Vertical" H 1000 4250 50  0001 C CNN
 F 3 "~" H 1000 4250 50  0001 C CNN
 	1    1000 4250
@@
 F 0 "C3" H 650 4600 50  0000 L CNN
 F 1 "20pF" H 550 4500 50  0000 L CNN
-F 2 "Capacitors_THT:C_Disc_D5.0mm_W2.5mm_P2.50mm" H 888 4400 50  0001 C CNN
+F 2 "Capacitor_THT:C_Disc_D5.0mm_W2.5mm_P2.50mm" H 888 4400 50  0001 C CNN
 F 3 "~" H 850 4550 50  0001 C CNN
 	1    850  4550
@@
 F 0 "C4" H 1250 4600 50  0000 L CNN
 F 1 "20pF" H 1250 4500 50  0000 L CNN
-F 2 "Capacitors_THT:C_Disc_D5.0mm_W2.5mm_P2.50mm" H 1188 4400 50  0001 C CNN
+F 2 "Capacitor_THT:C_Disc_D5.0mm_W2.5mm_P2.50mm" H 1188 4400 50  0001 C CNN
 F 3 "~" H 1150 4550 50  0001 C CNN
 	1    1150 4550
@@
 F 0 "C5" H 8215 3196 50  0000 L CNN
 F 1 "1uF" H 8215 3105 50  0000 L CNN
-F 2 "Capacitors_THT:C_Disc_D5.0mm_W2.5mm_P2.50mm" H 8138 3000 50  0001 C CNN
+F 2 "Capacitor_THT:C_Disc_D5.0mm_W2.5mm_P2.50mm" H 8138 3000 50  0001 C CNN
 F 3 "~" H 8100 3150 50  0001 C CNN
 	1    8100 3150
@@
 F 0 "C8" H 10415 3196 50  0000 L CNN
 F 1 "1uF" H 10415 3105 50  0000 L CNN
-F 2 "Capacitors_THT:C_Disc_D5.0mm_W2.5mm_P2.50mm" H 10338 3000 50  0001 C CNN
+F 2 "Capacitor_THT:C_Disc_D5.0mm_W2.5mm_P2.50mm" H 10338 3000 50  0001 C CNN
 F 3 "~" H 10300 3150 50  0001 C CNN
 	1    10300 3150
@@
 F 0 "C6" V 10200 3400 50  0000 C CNN
 F 1 "1uF" V 10300 3350 50  0000 C CNN
-F 2 "Capacitors_THT:C_Disc_D5.0mm_W2.5mm_P2.50mm" H 10288 3350 50  0001 C CNN
+F 2 "Capacitor_THT:C_Disc_D5.0mm_W2.5mm_P2.50mm" H 10288 3350 50  0001 C CNN
 F 3 "~" H 10250 3500 50  0001 C CNN
 	1    10250 3500
@@
 F 0 "C7" V 10200 3700 50  0000 C CNN
 F 1 "1uF" V 10300 3650 50  0000 C CNN
-F 2 "Capacitors_THT:C_Disc_D5.0mm_W2.5mm_P2.50mm" H 10288 3650 50  0001 C CNN
+F 2 "Capacitor_THT:C_Disc_D5.0mm_W2.5mm_P2.50mm" H 10288 3650 50  0001 C CNN
 F 3 "~" H 10250 3800 50  0001 C CNN
 	1    10250 3800
@@
 F 0 "R1" H 1770 1496 50  0000 L CNN
 F 1 "10K" H 1770 1405 50  0000 L CNN
-F 2 "Resistors_THT:R_Axial_DIN0207_L6.3mm_D2.5mm_P10.16mm_Horizontal" V 1630 1450 50  0001 C CNN
+F 2 "Resistor_THT:R_Axial_DIN0207_L6.3mm_D2.5mm_P10.16mm_Horizontal" V 1630 1450 50  0001 C CNN
 F 3 "~" H 1700 1450 50  0001 C CNN
 	1    1700 1450
@@
 F 0 "U1" H 2700 4700 50  0000 C CNN
 F 1 "PIC16F15345-IP" H 3100 4700 50  0000 C CNN
-F 2 "Housings_DIP:DIP-20_W7.62mm_LongPads" H 4700 4000 50  0001 C CNN
+F 2 "Package_DIP:DIP-20_W7.62mm_LongPads" H 4700 4000 50  0001 C CNN
 F 3 "http://ww1.microchip.com/downloads/en/DeviceDoc/40001865B.pdf" H 4700 4000 50  0001 C CNN
 	1    4700 4000
@@
 F 0 "D12" V 2339 5483 50  0000 R CNN
 F 1 "LED" V 2248 5483 50  0000 R CNN
-F 2 "LEDs:LED_D3.0mm" H 2300 5600 50  0001 C CNN
+F 2 "LED_THT:LED_D3.0mm" H 2300 5600 50  0001 C CNN
 F 3 "~" H 2300 5600 50  0001 C CNN
 	1    2300 5600
@@
 F 0 "R8" H 2370 5296 50  0000 L CNN
 F 1 "330R" H 2370 5205 50  0000 L CNN
-F 2 "Resistors_THT:R_Axial_DIN0207_L6.3mm_D2.5mm_P10.16mm_Horizontal" V 2230 5250 50  0001 C CNN
+F 2 "Resistor_THT:R_Axial_DIN0207_L6.3mm_D2.5mm_P10.16mm_Horizontal" V 2230 5250 50  0001 C CNN
 F 3 "~" H 2300 5250 50  0001 C CNN
 	1    2300 5250
