File: board/projector-screen-controller.sch (KiCad schematic (older format))
At the start: 9 parts, among them J2 MSTBVA-3-G, J3 MCV-3-G, J4 MCV-3-G, J5 MCV-3-G, J6 MSTBVA-6-G, J7 MCV-3-G

Commit message: Fix KiCad 4 footprints
* Update the Phoenix connectors with KiCad 5 footprints
Parts:
- J2: footprint Connectors_Phoenix:PhoenixContact_MSTBVA-G_03x5.00mm_Vertical -> Connector_Phoenix_MSTB:PhoenixContact_MSTBVA_2,5_3-G_1x03_P5.00mm_Vertical
- J3, J4, J5, J7: footprint Connectors_Phoenix:PhoenixContact_MCV-G_03x3.50mm_Vertical -> Connector_Phoenix_MC:PhoenixContact_MCV_1,5_3-G-3.5_1x03_P3.50mm_Vertical
- J6: footprint Connectors_Phoenix:PhoenixContact_MSTBVA-G_06x5.00mm_Vertical -> Connector_Phoenix_MSTB:PhoenixContact_MSTBVA_2,5_6-G_1x06_P5.00mm_Vertical
Changed lines of the file:
@@
 	1    0    0    -1
-$EndComp
-$Comp
-L Connector:Screw_Terminal_01x03 J2
-U 1 1 5D6FB32D
-P 1400 5300
-F 0 "J2" H 1550 5300 50  0000 C CNN
-F 1 "MSTBVA-3-G" H 1400 5050 50  0000 C CNN
-F 2 "Connectors_Phoenix:PhoenixContact_MSTBVA-G_03x5.00mm_Vertical" H 1400 5300 50  0001 C CNN
-F 3 "~" H 1400 5300 50  0001 C CNN
-F 4 "Phoenix Connect" H 1400 5300 50  0001 C CNN "mfr"
-F 5 "1924208" H 1400 5300 50  0001 C CNN "part#"
-	1    1400 5300
-	-1   0    0    -1
 $EndComp
 Wire Wire Line
@@
 F 0 "J3" H 1268 2367 50  0000 C CNN
 F 1 "MCV-3-G" H 1268 2276 50  0000 C CNN
-F 2 "Connectors_Phoenix:PhoenixContact_MCV-G_03x3.50mm_Vertical" H 1350 2050 50  0001 C CNN
+F 2 "Connector_Phoenix_MC:PhoenixContact_MCV_1,5_3-G-3.5_1x03_P3.50mm_Vertical" H 1350 2050 50  0001 C CNN
 F 3 "~" H 1350 2050 50  0001 C CNN
 	1    1350 2050
@@
 F 0 "J4" H 1268 2917 50  0000 C CNN
 F 1 "MCV-3-G" H 1268 2826 50  0000 C CNN
-F 2 "Connectors_Phoenix:PhoenixContact_MCV-G_03x3.50mm_Vertical" H 1350 2600 50  0001 C CNN
+F 2 "Connector_Phoenix_MC:PhoenixContact_MCV_1,5_3-G-3.5_1x03_P3.50mm_Vertical" H 1350 2600 50  0001 C CNN
 F 3 "~" H 1350 2600 50  0001 C CNN
 	1    1350 2600
@@
 F 0 "J5" H 1268 3467 50  0000 C CNN
 F 1 "MCV-3-G" H 1268 3376 50  0000 C CNN
-F 2 "Connectors_Phoenix:PhoenixContact_MCV-G_03x3.50mm_Vertical" H 1350 3150 50  0001 C CNN
+F 2 "Connector_Phoenix_MC:PhoenixContact_MCV_1,5_3-G-3.5_1x03_P3.50mm_Vertical" H 1350 3150 50  0001 C CNN
 F 3 "~" H 1350 3150 50  0001 C CNN
 	1    1350 3150
@@
 F 0 "J6" H 9930 2542 50  0000 L CNN
 F 1 "MSTBVA-6-G" H 9930 2451 50  0000 L CNN
-F 2 "Connectors_Phoenix:PhoenixContact_MSTBVA-G_06x5.00mm_Vertical" H 9850 2550 50  0001 C CNN
+F 2 "Connector_Phoenix_MSTB:PhoenixContact_MSTBVA_2,5_6-G_1x06_P5.00mm_Vertical" H 9850 2550 50  0001 C CNN
 F 3 "~" H 9850 2550 50  0001 C CNN
 	1    9850 2550
@@
 F 0 "J7" H 1268 4017 50  0000 C CNN
 F 1 "MCV-3-G" H 1268 3926 50  0000 C CNN
-F 2 "Connectors_Phoenix:PhoenixContact_MCV-G_03x3.50mm_Vertical" H 1350 3700 50  0001 C CNN
+F 2 "Connector_Phoenix_MC:PhoenixContact_MCV_1,5_3-G-3.5_1x03_P3.50mm_Vertical" H 1350 3700 50  0001 C CNN
 F 3 "~" H 1350 3700 50  0001 C CNN
 	1    1350 3700
@@
 	6350 5650 6350 6050
 Connection ~ 6100 5650
+$Comp
+L Connector:Screw_Terminal_01x03 J2
+U 1 1 5D6FB32D
+P 1400 5300
+F 0 "J2" H 1550 5300 50  0000 C CNN
+F 1 "MSTBVA-3-G" H 1400 5050 50  0000 C CNN
+F 2 "Connector_Phoenix_MSTB:PhoenixContact_MSTBVA_2,5_3-G_1x03_P5.00mm_Vertical" H 1400 5300 50  0001 C CNN
+F 3 "~" H 1400 5300 50  0001 C CNN
+F 4 "Phoenix Connect" H 1400 5300 50  0001 C CNN "mfr"
+F 5 "1924208" H 1400 5300 50  0001 C CNN "part#"
+	1    1400 5300
+	-1   0    0    -1
+$EndComp
 $EndSCHEMATC

Commit message: Fix channel 2 button reversal
* The hierarchical schematic pins for channel 2 buttons were reversed in the
  root schematic. Correct this, and add board revision logic to the firmware so
  board versions can be targeted by the build.
Connections:
- net MCU/BUT2_DN: now also J7.2 (Pin_2); no longer J7.3 (Pin_3)
- net MCU/BUT2_UP: now also J7.3 (Pin_3); no longer J7.2 (Pin_2)
Changed lines of the file:
@@
 Sheet 1 4
 Title "Projector Screen Controller"
-Date "2019-09-07"
+Date "2019-09-13"
 Rev "0.2"
 Comp "Flirble Open Source"
@@
 F10 "BUT1_UP" I L 3750 3250 50
 F11 "BUT1_DN" I L 3750 3150 50
-F12 "BUT2_UP" I L 3750 3350 50
-F13 "BUT2_DN" I L 3750 3450 50
+F12 "BUT2_UP" I L 3750 3450 50
+F13 "BUT2_DN" I L 3750 3350 50
 $EndSheet
 $Sheet
