File: board/Relay.sch (KiCad schematic (older format))
At the start: 18 parts, among them K1 JS1-12V-F, K2 JS1-12V-F, K3 JS1-12V-F, K4 JS1-12V-F, U4 ULN2003A

Commit message: Add/correct a bunch of part numbers
Parts:
- K1, K2, K3, K4: Src1 (none) -> Mouser; Src1 Part (none) -> 769-JS1-12V-F; Src1 URL (none) -> https://www.mouser.com/ProductDetail/769-JS1-12V-F; mfr (none) -> Panasonic; mpn (none) -> JS1-12V-F
- U4: Src1 (none) -> Mouser; Src1 Part (none) -> 511-ULN2003A; Src1 URL (none) -> https://www.mouser.com/ProductDetail/511-ULN2003A; mfr (none) -> ST; mpn (none) -> ULN2003A
Changed lines of the file:
@@
 F 2 "Package_DIP:DIP-16_W7.62mm_LongPads" H 3200 2150 50  0001 L CNN
 F 3 "http://www.ti.com/lit/ds/symlink/uln2003a.pdf" H 3250 2500 50  0001 C CNN
+F 4 "ST" H 3150 2700 50  0001 C CNN "mfr"
+F 5 "ULN2003A" H 3150 2700 50  0001 C CNN "mpn"
+F 6 "Mouser" H 3150 2700 50  0001 C CNN "Src1"
+F 7 "511-ULN2003A" H 3150 2700 50  0001 C CNN "Src1 Part"
+F 8 "https://www.mouser.com/ProductDetail/511-ULN2003A" H 3150 2700 50  0001 C CNN "Src1 URL"
 	1    3150 2700
 	1    0    0    -1
@@
 F 2 "Relay_THT:Relay_SPDT_SANYOU_SRD_Series_Form_C" H 6900 2000 50  0001 L CNN
 F 3 "https://www3.panasonic.biz/ac/cdn/e/control/relay/power/catalog/mech_eng_js.pdf" H 6450 2050 50  0001 C CNN
+F 4 "Panasonic" H 6450 2050 50  0001 C CNN "mfr"
+F 5 "JS1-12V-F" H 6450 2050 50  0001 C CNN "mpn"
+F 6 "Mouser" H 6450 2050 50  0001 C CNN "Src1"
+F 7 "769-JS1-12V-F" H 6450 2050 50  0001 C CNN "Src1 Part"
+F 8 "https://www.mouser.com/ProductDetail/769-JS1-12V-F" H 6450 2050 50  0001 C CNN "Src1 URL"
 	1    6450 2050
 	1    0    0    -1
@@
 F 2 "Relay_THT:Relay_SPDT_SANYOU_SRD_Series_Form_C" H 6900 2950 50  0001 L CNN
 F 3 "https://www3.panasonic.biz/ac/cdn/e/control/relay/power/catalog/mech_eng_js.pdf" H 6450 3000 50  0001 C CNN
+F 4 "https://www.mouser.com/ProductDetail/769-JS1-12V-F" H 6450 3000 50  0001 C CNN "Src1 URL"
+F 5 "Panasonic" H 6450 3000 50  0001 C CNN "mfr"
+F 6 "JS1-12V-F" H 6450 3000 50  0001 C CNN "mpn"
+F 7 "Mouser" H 6450 3000 50  0001 C CNN "Src1"
+F 8 "769-JS1-12V-F" H 6450 3000 50  0001 C CNN "Src1 Part"
 	1    6450 3000
 	1    0    0    -1
@@
 F 2 "Relay_THT:Relay_SPDT_SANYOU_SRD_Series_Form_C" H 6900 3950 50  0001 L CNN
 F 3 "https://www3.panasonic.biz/ac/cdn/e/control/relay/power/catalog/mech_eng_js.pdf" H 6450 4000 50  0001 C CNN
+F 4 "https://www.mouser.com/ProductDetail/769-JS1-12V-F" H 6450 4000 50  0001 C CNN "Src1 URL"
+F 5 "Panasonic" H 6450 4000 50  0001 C CNN "mfr"
+F 6 "JS1-12V-F" H 6450 4000 50  0001 C CNN "mpn"
+F 7 "Mouser" H 6450 4000 50  0001 C CNN "Src1"
+F 8 "769-JS1-12V-F" H 6450 4000 50  0001 C CNN "Src1 Part"
 	1    6450 4000
 	1    0    0    -1
@@
 F 2 "Relay_THT:Relay_SPDT_SANYOU_SRD_Series_Form_C" H 6900 5000 50  0001 L CNN
 F 3 "https://www3.panasonic.biz/ac/cdn/e/control/relay/power/catalog/mech_eng_js.pdf" H 6450 5050 50  0001 C CNN
+F 4 "Panasonic" H 6450 5050 50  0001 C CNN "mfr"
+F 5 "JS1-12V-F" H 6450 5050 50  0001 C CNN "mpn"
+F 6 "Mouser" H 6450 5050 50  0001 C CNN "Src1"
+F 7 "769-JS1-12V-F" H 6450 5050 50  0001 C CNN "Src1 Part"
+F 8 "https://www.mouser.com/ProductDetail/769-JS1-12V-F" H 6450 5050 50  0001 C CNN "Src1 URL"
 	1    6450 5050
 	1    0    0    -1

Commit message: First pass at input protection for buttons
* Schottky diodes & capacitors to limit and smooth the inputs.
* Relies on the WPU of the MCU to provide a charge for the C (possibly
  a bad idea, will see).
* Had to move a bunch of stuff to make room and make sure the ground paths
  were sensible.
* Update all the disc capacitors to the Kicad 5 footprint.
Parts:
- C13: footprint Capacitor_THT:C_Disc_D5.0mm_W2.5mm_P2.50mm -> Capacitors_THT:C_Disc_D5.0mm_W2.5mm_P2.50mm
- D10, D11, D8, D9: footprint LED_THT:LED_D3.0mm -> LEDs:LED_D3.0mm
Changed lines of the file:
@@
 F 0 "D8" V 1200 3400 50  0000 R CNN
 F 1 "LED" V 1100 3400 50  0000 R CNN
-F 2 "LED_THT:LED_D3.0mm" H 1150 3450 50  0001 C CNN
+F 2 "LEDs:LED_D3.0mm" H 1150 3450 50  0001 C CNN
 F 3 "~" H 1150 3450 50  0001 C CNN
 	1    1150 3450
@@
 F 0 "D9" V 1450 3400 50  0000 R CNN
 F 1 "LED" V 1350 3400 50  0000 R CNN
-F 2 "LED_THT:LED_D3.0mm" H 1400 3450 50  0001 C CNN
+F 2 "LEDs:LED_D3.0mm" H 1400 3450 50  0001 C CNN
 F 3 "~" H 1400 3450 50  0001 C CNN
 	1    1400 3450
@@
 F 0 "D10" V 1700 3400 50  0000 R CNN
 F 1 "LED" V 1600 3400 50  0000 R CNN
-F 2 "LED_THT:LED_D3.0mm" H 1650 3450 50  0001 C CNN
+F 2 "LEDs:LED_D3.0mm" H 1650 3450 50  0001 C CNN
 F 3 "~" H 1650 3450 50  0001 C CNN
 	1    1650 3450
@@
 F 0 "D11" V 1950 3400 50  0000 R CNN
 F 1 "LED" V 1850 3400 50  0000 R CNN
-F 2 "LED_THT:LED_D3.0mm" H 1900 3450 50  0001 C CNN
+F 2 "LEDs:LED_D3.0mm" H 1900 3450 50  0001 C CNN
 F 3 "~" H 1900 3450 50  0001 C CNN
 	1    1900 3450
@@
 F 0 "C13" H 3815 3396 50  0000 L CNN
 F 1 "0.1uF" H 3815 3305 50  0000 L CNN
-F 2 "Capacitor_THT:C_Disc_D5.0mm_W2.5mm_P2.50mm" H 3738 3200 50  0001 C CNN
+F 2 "Capacitors_THT:C_Disc_D5.0mm_W2.5mm_P2.50mm" H 3738 3200 50  0001 C CNN
 F 3 "~" H 3700 3350 50  0001 C CNN
 	1    3700 3350
